File: sch/max-power/max-power.sch (KiCad schematic (older format))
At the start: 44 parts, among them P1 CONN_01X09, P10 CONN_01X02, P2 CONN_01X09, P3 CONN_01X09, P4 CONN_01X04, P5 CONN_02X06, P6 CONN_02X04, P7 CONN_01X04, P8 CONN_02X05, P9 CONN_01X09, Q1 2N7002, SW1 SW_PUSH, U1 ATX-PWR-24P

Commit message: Initial placement of footprints.
Parts:
- added P7: CONN_01X02, Sockets_MOLEX_KK-System:Socket_MOLEX-KK-RM2-54mm_Lock_2pin_straight, symbol CONN_01X02
- C1: renamed from C5; footprint Capacitors_ThroughHole:C_Radial_D10_L13_P5 -> Capacitors_THT:C_Radial_D10_L13_P5; manf# (none) -> 25PX680MEFC10X12.5
- C10: renamed from C12; footprint Capacitors_ThroughHole:C_Radial_D10_L13_P5 -> Capacitors_THT:C_Radial_D10_L13_P5
- C11: renamed from C16; manf# (none) -> CL21B104MBCNNNC
- C12: renamed from C8; footprint Capacitors_ThroughHole:C_Radial_D10_L13_P5 -> Capacitors_THT:C_Radial_D10_L13_P5
- C14: renamed from C13; footprint Capacitors_ThroughHole:C_Radial_D10_L13_P5 -> Capacitors_THT:C_Radial_D10_L13_P5
- C16: renamed from C1; footprint Capacitors_ThroughHole:C_Radial_D5_L11_P2 -> Capacitors_THT:C_Radial_D5_L11_P2
- C17: renamed from C2; footprint Capacitors_ThroughHole:C_Radial_D5_L11_P2 -> Capacitors_THT:C_Radial_D5_L11_P2
- C18: renamed from C3; footprint Capacitors_ThroughHole:C_Radial_D5_L11_P2 -> Capacitors_THT:C_Radial_D5_L11_P2
- C19: renamed from C4; footprint Capacitors_ThroughHole:C_Radial_D5_L11_P2 -> Capacitors_THT:C_Radial_D5_L11_P2
- C2: renamed from C15; footprint Capacitors_ThroughHole:C_Radial_D10_L13_P5 -> Capacitors_THT:C_Radial_D10_L13_P5; manf# (none) -> ESC687M010AH1AA
- C20: renamed from C6; footprint Capacitors_ThroughHole:C_Radial_D5_L11_P2 -> Capacitors_THT:C_Radial_D5_L11_P2
- C21: renamed from C9; footprint Capacitors_ThroughHole:C_Radial_D10_L13_P5 -> Capacitors_THT:C_Radial_D5_L11_P2
- C24: renamed from C14; footprint Capacitors_ThroughHole:C_Radial_D10_L13_P5 -> Capacitors_THT:C_Radial_D5_L11_P2; manf# (none) -> ESK107M025AC3AA
- C25: renamed from C18; footprint Capacitors_ThroughHole:C_Radial_D10_L13_P5 -> Capacitors_THT:C_Radial_D5_L11_P2
- C26: renamed from C20; footprint Capacitors_ThroughHole:C_Radial_D10_L13_P5 -> Capacitors_THT:C_Radial_D5_L11_P2
- C27: renamed from C21; footprint Capacitors_ThroughHole:C_Radial_D10_L13_P5 -> Capacitors_THT:C_Radial_D5_L11_P2
- C3: renamed from C19; footprint Capacitors_ThroughHole:C_Radial_D10_L13_P5 -> Capacitors_THT:C_Radial_D10_L13_P5
- C4: renamed from C22; footprint Capacitors_ThroughHole:C_Radial_D10_L13_P5 -> Capacitors_THT:C_Radial_D10_L13_P5
- C5: renamed from C23; footprint Capacitors_ThroughHole:C_Radial_D10_L13_P5 -> Capacitors_THT:C_Radial_D5_L11_P2
- C6: renamed from C24; footprint Capacitors_ThroughHole:C_Radial_D10_L13_P5 -> Capacitors_THT:C_Radial_D5_L11_P2; manf# (none) -> ESK107M010AC3AA
- C7: renamed from C25; footprint Capacitors_ThroughHole:C_Radial_D10_L13_P5 -> Capacitors_THT:C_Radial_D5_L11_P2
- C8: renamed from C7; footprint Capacitors_ThroughHole:C_Radial_D10_L13_P5 -> Capacitors_THT:C_Radial_D10_L13_P5
- P1: renamed from P4; footprint (none) -> Additional connectors:conn_hdd_15-24-4449; manf# (none) -> 0015244449
- P12: renamed from P5; footprint (none) -> doragasu:TERM_BLOCK_6x2_5.08
- P13: renamed from P6; footprint (none) -> doragasu:TERM_BLOCK_4x2_5.08
- P2: renamed from P7; footprint (none) -> Additional connectors:conn_hdd_15-24-4449; manf# (none) -> 0015244449
- P3: renamed from U1; footprint (none) -> doragasu:ATX_PWR_CON; manf# (none) -> 0442060007
- P4: renamed from P8; footprint Connect:IDC_Header_Straight_10pins -> Connectors:IDC_Header_Straight_10pins
- P6: renamed from P10; footprint (none) -> Sockets_MOLEX_KK-System:Socket_MOLEX-KK-RM2-54mm_Lock_2pin_straight
- SW1: footprint Buttons_Switches_ThroughHole:SW_Tactile_SPST_Angled -> Buttons_Switches_THT:SW_Tactile_SPST_Angled
- renumbered C11 to C13, C17 to C15, C10 to C9, P3 to P10, P9 to P5, P1 to P8, P2 to P9, R3 to R2, R2 to R3, R5 to R4, R4 to R5
Connections:
- net GND: now also P7.2 (P2)
- net PWR_SW: now also P7.1 (P1)
- no-connect marks 17 -> 18
Other:
- moved on the sheet: C24, C25, C26, C27, P12, P13

Commit message: Routed PCB.
Parts:
- added P11: CONN_01X02, Sockets_MOLEX_KK-System:Socket_MOLEX-KK-RM3-96mm_Lock_2pin_straight, symbol CONN_01X02
- SW1: footprint Buttons_Switches_THT:SW_Tactile_SPST_Angled -> Buttons_Switches_THT:SW_PUSH_SMALL
Connections:
- net +12V: now also P12.10 (P10), P12.12 (P12), P12.2 (P2), P12.4 (P4), P12.6 (P6), P12.8 (P8); no longer P12.1 (P1), P12.11 (P11), P12.3 (P3), P12.5 (P5), P12.7 (P7), P12.9 (P9)
- net +3V3: now also P13.2 (P2), P13.4 (P4), P13.6 (P6), P13.8 (P8); no longer P13.1 (P1), P13.3 (P3), P13.5 (P5), P13.7 (P7)
- net +5V: now also P11.1 (P1)
- net GND: now also P12.1 (P1), P12.11 (P11), P12.3 (P3), P12.5 (P5), P12.7 (P7), P12.9 (P9), P13.1 (P1), P13.3 (P3), P13.5 (P5), P13.7 (P7), P11.2 (P2); no longer P12.10 (P10), P12.12 (P12), P12.2 (P2), P12.4 (P4), P12.6 (P6), P12.8 (P8), P13.2 (P2), P13.4 (P4), P13.6 (P6), P13.8 (P8)
- net PS_ON: now also P4.6 (P6); no longer P4.5 (P5)
- net PWR_SW: now also P4.5 (P5); no longer P4.6 (P6)
Other:
- moved on the sheet: D1, P7, R4, R5, SW1
Changed lines of the file:
@@
 	-1   0    0    1
 $EndComp
-Text Label 6150 2750 2    60   ~ 0
+Text Label 5900 2750 2    60   ~ 0
 PS_ON
 $Comp
 L SW_PUSH SW1
 U 1 1 586B5888
-P 5650 3700
-F 0 "SW1" V 5604 3818 50  0000 L CNN
-F 1 "SW_PUSH" V 5695 3818 50  0000 L CNN
-F 2 "Buttons_Switches_THT:SW_Tactile_SPST_Angled" H 5650 3700 50  0001 C CNN
-F 3 "" H 5650 3700 50  0000 C CNN
-	1    5650 3700
+P 5500 3700
+F 0 "SW1" V 5454 3818 50  0000 L CNN
+F 1 "SW_PUSH" V 5545 3818 50  0000 L CNN
+F 2 "Buttons_Switches_THT:SW_PUSH_SMALL" H 5500 3700 50  0001 C CNN
+F 3 "" H 5500 3700 50  0000 C CNN
+	1    5500 3700
 	0    1    1    0
 $EndComp
@@
 L R R5
 U 1 1 586B59A3
-P 5650 3200
-F 0 "R5" H 5720 3246 50  0000 L CNN
-F 1 "R" H 5720 3155 50  0000 L CNN
-F 2 "Resistors_SMD:R_0805" V 5580 3200 50  0001 C CNN
-F 3 "" H 5650 3200 50  0000 C CNN
-	1    5650 3200
+P 5500 3200
+F 0 "R5" H 5570 3246 50  0000 L CNN
+F 1 "R" H 5570 3155 50  0000 L CNN
+F 2 "Resistors_SMD:R_0805" V 5430 3200 50  0001 C CNN
+F 3 "" H 5500 3200 50  0000 C CNN
+	1    5500 3200
 	1    0    0    -1
 $EndComp
@@
 L GND #PWR020
 U 1 1 586B5AE5
-P 5650 4000
-F 0 "#PWR020" H 5650 3750 50  0001 C CNN
-F 1 "GND" H 5655 3827 50  0001 C CNN
-F 2 "" H 5650 4000 50  0000 C CNN
-F 3 "" H 5650 4000 50  0000 C CNN
-	1    5650 4000
-	1    0    0    -1
-$EndComp
-Text Label 6150 3400 2    60   ~ 0
+P 5500 4000
+F 0 "#PWR020" H 5500 3750 50  0001 C CNN
+F 1 "GND" H 5505 3827 50  0001 C CNN
+F 2 "" H 5500 4000 50  0000 C CNN
+F 3 "" H 5500 4000 50  0000 C CNN
+	1    5500 4000
+	1    0    0    -1
+$EndComp
+Text Label 6000 3400 2    60   ~ 0
 PWR_SW
 $Comp
@@
 L LED D1
 U 1 1 586BE47F
-P 6200 2950
-F 0 "D1" H 6200 3050 50  0000 C CNN
-F 1 "LED" H 6200 3150 50  0000 C CNN
-F 2 "LEDs:LED-5MM" H 6200 2950 50  0001 C CNN
-F 3 "" H 6200 2950 50  0000 C CNN
-	1    6200 2950
+P 6050 2950
+F 0 "D1" H 6050 3050 50  0000 C CNN
+F 1 "LED" H 6050 3150 50  0000 C CNN
+F 2 "LEDs:LED-5MM" H 6050 2950 50  0001 C CNN
+F 3 "" H 6050 2950 50  0000 C CNN
+	1    6050 2950
 	-1   0    0    1
 $EndComp
@@
 L R R4
 U 1 1 586BE726
-P 5850 2950
-F 0 "R4" H 5920 2996 50  0000 L CNN
-F 1 "R" H 5920 2905 50  0000 L CNN
-F 2 "Resistors_SMD:R_0805" V 5780 2950 50  0001 C CNN
-F 3 "" H 5850 2950 50  0000 C CNN
-	1    5850 2950
+P 5700 2950
+F 0 "R4" H 5770 2996 50  0000 L CNN
+F 1 "R" H 5770 2905 50  0000 L CNN
+F 2 "Resistors_SMD:R_0805" V 5630 2950 50  0001 C CNN
+F 3 "" H 5700 2950 50  0000 C CNN
+	1    5700 2950
 	0    1    1    0
 $EndComp
-Text Label 6150 2850 2    60   ~ 0
+Text Label 6000 2850 2    60   ~ 0
 3.3VPI
 $Comp
@@
 F 3 "" H 5300 5000 50  0000 C CNN
 	1    5300 6200
-	1    0    0    -1
+	-1   0    0    -1
 $EndComp
 $Comp
@@
 F 3 "" H 6300 5000 50  0000 C CNN
 	1    6300 6200
-	1    0    0    -1
+	-1   0    0    -1
 $EndComp
 $Comp
@@
 L CONN_01X02 P7
 U 1 1 5870F5C1
-P 5200 3700
-F 0 "P7" H 5250 3750 50  0000 L CNN
-F 1 "CONN_01X02" H 5250 3650 50  0000 L CNN
-F 2 "Sockets_MOLEX_KK-System:Socket_MOLEX-KK-RM2-54mm_Lock_2pin_straight" H 5200 3700 50  0001 C CNN
-F 3 "" H 5200 3700 50  0000 C CNN
-	1    5200 3700
+P 5050 3700
+F 0 "P7" H 5100 3750 50  0000 L CNN
+F 1 "CONN_01X02" H 5100 3650 50  0000 L CNN
+F 2 "Sockets_MOLEX_KK-System:Socket_MOLEX-KK-RM2-54mm_Lock_2pin_straight" H 5050 3700 50  0001 C CNN
+F 3 "" H 5050 3700 50  0000 C CNN
+	1    5050 3700
 	-1   0    0    -1
 $EndComp
@@
 Connection ~ 4900 3150
 Wire Wire Line
-	5600 2750 6400 2750
-Wire Wire Line
-	5650 3350 5650 3400
-Wire Wire Line
-	5400 3400 7050 3400
-Connection ~ 5650 3400
+	5600 2750 6050 2750
+Wire Wire Line
+	5500 3350 5500 3400
+Wire Wire Line
+	5250 3400 6300 3400
+Connection ~ 5500 3400
 Wire Wire Line
 	6350 2500 6350 2650
@@
 Connection ~ 6350 2550
 Wire Wire Line
-	5650 2850 5650 3050
-Wire Wire Line
-	5650 2850 6400 2850
+	5500 2850 5500 3050
+Wire Wire Line
+	5500 2850 6400 2850
 Wire Wire Line
 	6950 2550 6950 3050
@@
 Connection ~ 6950 2950
 Wire Wire Line
-	5700 2950 5650 2950
-Connection ~ 5650 2950
+	5550 2950 5500 2950
+Connection ~ 5500 2950
 Wire Wire Line
 	6900 2750 7050 2750
-Wire Wire Line
-	7050 2750 7050 3400
 Wire Wire Line
 	5550 6050 5600 6050
@@
 	5350 1400 5550 1400
 Wire Wire Line
-	6400 2950 6400 3150
-Connection ~ 6400 2950
-Wire Wire Line
-	6400 3250 6000 3250
-Wire Wire Line
-	6000 3250 6000 2950
-Connection ~ 6000 2950
-Wire Wire Line
-	5400 3400 5400 3650
-Wire Wire Line
-	5400 3750 5400 4000
-Wire Wire Line
-	5400 4000 5650 4000
-Connection ~ 5650 4000
+	6400 3250 5850 3250
+Wire Wire Line
+	5850 3250 5850 2950
+Connection ~ 5850 2950
+Wire Wire Line
+	5250 3400 5250 3650
+Wire Wire Line
+	5250 3750 5250 4000
+Wire Wire Line
+	5250 4000 5500 4000
+Connection ~ 5500 4000
 Wire Wire Line
 	7400 2900 7550 2900
@@
 	1    0    0    -1
 $EndComp
+$Comp
+L CONN_01X02 P11
+U 1 1 5871FA45
+P 6700 4000
+F 0 "P11" H 6778 4041 50  0000 L CNN
+F 1 "CONN_01X02" H 6778 3950 50  0000 L CNN
+F 2 "Sockets_MOLEX_KK-System:Socket_MOLEX-KK-RM3-96mm_Lock_2pin_straight" H 6700 4000 50  0001 C CNN
+F 3 "" H 6700 4000 50  0000 C CNN
+	1    6700 4000
+	1    0    0    -1
+$EndComp
+$Comp
+L +5V #PWR065
+U 1 1 587201AF
+P 6450 3900
+F 0 "#PWR065" H 6450 3750 50  0001 C CNN
+F 1 "+5V" H 6400 4050 50  0000 C CNN
+F 2 "" H 6450 3900 50  0000 C CNN
+F 3 "" H 6450 3900 50  0000 C CNN
+	1    6450 3900
+	1    0    0    -1
+$EndComp
+Wire Wire Line
+	6450 3900 6450 3950
+Wire Wire Line
+	6450 3950 6500 3950
+$Comp
+L GND #PWR066
+U 1 1 58720404
+P 6450 4100
+F 0 "#PWR066" H 6450 3850 50  0001 C CNN
+F 1 "GND" H 6455 3927 50  0001 C CNN
+F 2 "" H 6450 4100 50  0000 C CNN
+F 3 "" H 6450 4100 50  0000 C CNN
+	1    6450 4100
+	1    0    0    -1
+$EndComp
+Wire Wire Line
+	6450 4100 6450 4050
+Wire Wire Line
+	6450 4050 6500 4050
+Wire Wire Line
+	7050 2750 7050 2300
+Wire Wire Line
+	7050 2300 6050 2300
+Wire Wire Line
+	6050 2300 6050 2750
+Wire Wire Line
+	6300 3400 6300 2750
+Wire Wire Line
+	6300 2750 6400 2750
+Wire Wire Line
+	6250 2950 6400 2950
+Wire Wire Line
+	6400 2950 6400 3150
+Connection ~ 6400 2950
 $EndSCHEMATC
